File: Hardware/Frontplate/Frontplate.kicad_pcb (KiCad board)
At the start: 2 copper layers, 78 x 27 mm, 5 parts

Commit message: First working version, with 12-lead recording
Other:
- board text added: "JLCJLCJLCJLC"
Changed lines of the file:
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@@
       (outputformat 1)
       (mirror false)
-      (drillshape 1)
+      (drillshape 0)
       (scaleselection 1)
-      (outputdirectory "")
+      (outputdirectory "Output/Gerbers")
     )
   )
@@
   (gr_line (start 139.2 73) (end 139.2 82.2)
     (stroke (width 0.15) (type default)) (layer "User.9"))
+  (gr_text "JLCJLCJLCJLC" (at 171.3 99.8) (layer "B.SilkS")
+    (effects (font (size 0.7 0.7) (thickness 0.15)) (justify left bottom mirror))
+  )
   (gr_text "SimpleECG" (at 128 80) (layer "F.Mask")
     (effects (font (face "Futura") (size 3 3) (thickness 0.15)) (justify left bottom))
