File: Hardware/PCB/SimpleECG_v0.kicad_pcb (KiCad board)
At the start: 4 copper layers, 119 x 74 mm, 153 parts, among them J1 USB_C_Receptacle_USB2.0, J2 Conn_01x15, J3 Micro_SD_Card, SW1 SW_Push, U1 STM32F103CBTx, U2 AMS1117-3.3, U3 ADS1298xPAG, U4 AMS1117-3.3, Y1 8 MHz

Commit message: First working version, with 12-lead recording
Routing:
- net GND: track 96.7 -> 103.6 mm
Changed lines of the file:
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@@
   (dimension (type aligned) (layer "Cmts.User")
     (pts (xy 172.3 19) (xy 172.3 93))
-    (height -7.8)
-    (gr_text "74.0000 mm" (at 178.95 56 90) (layer "Cmts.User")
+    (height -6)
+    (gr_text "74.0000 mm" (at 177.3 56 90) (layer "Cmts.User")
       (effects (font (size 1 1) (thickness 0.15)))
     )
     (format (prefix "") (suffix "") (units 3) (units_format 1) (precision 4))
-    (style (thickness 0.15) (arrow_length 1.27) (text_position_mode 0) (extension_height 0.58642) (extension_offset 0.5) keep_text_aligned)
+    (style (thickness 0.15) (arrow_length 1.27) (text_position_mode 2) (extension_height 0.58642) (extension_offset 0.5) keep_text_aligned)
   )
   (dimension (type aligned) (layer "Cmts.User")
     (pts (xy 53.3 19) (xy 172.3 19))
-    (height -6.1)
-    (gr_text "119.0000 mm" (at 112.8 11.75) (layer "Cmts.User")
+    (height -5)
+    (gr_text "119.0000 mm" (at 112.8 15) (layer "Cmts.User")
       (effects (font (size 1 1) (thickness 0.15)))
     )
     (format (prefix "") (suffix "") (units 3) (units_format 1) (precision 4))
-    (style (thickness 0.15) (arrow_length 1.27) (text_position_mode 0) (extension_height 0.58642) (extension_offset 0.5) keep_text_aligned)
+    (style (thickness 0.15) (arrow_length 1.27) (text_position_mode 2) (extension_height 0.58642) (extension_offset 0.5) keep_text_aligned)
   )
   (segment (start 129.79917 52.5945) (end 129.33 52.12533) (width 0.2) (layer "F.Cu") (net 1))
@@
   (segment (start 93.05 50.2) (end 93.8 50.2) (width 0.5) (layer "F.Cu") (net 2))
   (segment (start 99.3 51) (end 99.3 50.1) (width 0.2) (layer "F.Cu") (net 2))
+  (segment (start 63.2375 83.0625) (end 66 80.3) (width 0.25) (layer "F.Cu") (net 2))
   (segment (start 103.8 62.325) (end 103.8 61.2) (width 0.2) (layer "F.Cu") (net 2))
   (segment (start 86.01825 57.19375) (end 86.012 57.2) (width 0.2) (layer "F.Cu") (net 2))
@@
   (segment (start 107.15 63.6) (end 108.2 63.6) (width 1) (layer "F.Cu") (net 2))
   (segment (start 74.5625 51.89375) (end 74.2125 52.24375) (width 0.5) (layer "F.Cu") (net 2))
+  (segment (start 60.3 83.0625) (end 63.2375 83.0625) (width 0.25) (layer "F.Cu") (net 2))
   (segment (start 86.825 34.39375) (end 86.01825 34.39375) (width 0.2) (layer "F.Cu") (net 2))
   (segment (start 86.825 68.69375) (end 86.01825 68.69375) (width 0.2) (layer "F.Cu") (net 2))
